Commit message: Q1 Wheel hardware sheet: CubeMars motors, MTi-630 IMU, 40 kg URDF, X2 reference clip
- config/q1_wheel_components.yaml: CubeMars AKE90-8 / AK10-9 / AK45-36 / AK45-10 datasheet
  numbers, 24-joint -> SKU map from the BI2 slide, IMU placement, CAN 200 Hz, wheel r=0.1 m
- tools/build_urdf.py: generates urdf/wheel_humanoid.urdf from the structural CAD URDF:
  stator masses on the parent links, 40.0 kg total, neck/wrist/gripper joints (24 DoF),
  imu_link on the pelvis at hip-axis height, SKU torque/speed limits, zero PhysX friction
- docs/reference: Lingxi X2 skate clip (1:45-2:00) + MediaPipe pose angles / Q1 keyframe
- tools/x2_pose_extract.py: MediaPipe PoseLandmarker -> sagittal joint angles -> Q1 mapping
- wheel_humanoid_lab.actuators.CubeMarsActuator: voltage/current limited BLDC plant with
  in-actuator friction, command delay, bus sag and restore-then-sample DR
- assets: Q1_WHEEL_CUBEMARS_CFG (actuators grouped by SKU), 24-D joint contract (q1_spec)
- tasks/skate: Isaac-Q1-Skate-v0 (92-D actor obs, 24-D action, IMU obs with delay/tilt,
  swizzle/lean/arms-back/micro-lift rewards, 6-stage curriculum, non-accumulating CoM DR)
- tests/test_skate_contract.py: obs/action/actuator contract test (passes, 4 envs)

File: urdf/wheel_humanoid.urdf (robot description, URDF)
Before this commit: robot wheel_humanoid, 22 links, 21 joints
Links:
- added link head_link, mass 0.1500; collision cylinder length=0.0565 radius=0.0275; visual cylinder length=0.0565 radius=0.0275
- added link imu_link, mass 0.0550; visual box size=0.0573 0.0416 0.0236
- added link l_gripper_link, mass 0.2000; collision cylinder length=0.0452 radius=0.0265; visual cylinder length=0.0452 radius=0.0265
- added link l_wrist_link, mass 0.3820; collision cylinder length=0.0452 radius=0.0265; visual cylinder length=0.0452 radius=0.0265
- added link r_gripper_link, mass 0.2000; collision cylinder length=0.0452 radius=0.0265; visual cylinder length=0.0452 radius=0.0265
- added link r_wrist_link, mass 0.3820; collision cylinder length=0.0452 radius=0.0265; visual cylinder length=0.0452 radius=0.0265
- link l_elbow_link: mass 0.1871 -> 0.4363
- link l_hip_pitch_link: mass 0.5906 -> 1.9503
- link l_knee_roller_link: mass 0.1714 -> 0.1597
- link l_shin_link: mass 1.1424 -> 2.0045
- link l_shoulder_pitch_link: mass 0.4382 -> 1.3483
- link l_shoulder_roll_link: mass 0.4578 -> 1.3666
- link l_shoulder_yaw_link: mass 0.4871 -> 1.3939
- link l_thigh_link: mass 0.9136 -> 2.2513
- link l_wheel_link: mass 1.3349 -> 1.2439
- link pelvis: mass 1.6502 -> 5.2777
- link r_elbow_link: mass 0.1871 -> 0.4363
- link r_hip_pitch_link: mass 0.5860 -> 1.9460
- link r_knee_roller_link: mass 0.1714 -> 0.1597
- link r_shin_link: mass 1.1424 -> 2.0045
- link r_shoulder_pitch_link: mass 0.4381 -> 1.3482
- link r_shoulder_roll_link: mass 0.4578 -> 1.3666
- link r_shoulder_yaw_link: mass 0.4871 -> 1.3939
- link r_thigh_link: mass 0.9189 -> 2.2562
- link r_wheel_link: mass 1.3349 -> 1.2439
- link torso: mass 5.1562 -> 7.0335
- link waist_roll_link: mass 0.0284 -> 0.9665
- link waist_yaw_link: mass 0.1108 -> 1.0432
Joints:
- added joint imu_joint: type fixed, parent pelvis, child imu_link, origin xyz=0.0 0.0 -0.1267 rpy=0.0 0.0 0.0
- added joint l_gripper_joint: type revolute, parent l_wrist_link, child l_gripper_link, origin xyz=0.0 0.0 -0.05 rpy=0.0 0.0 0.0, axis 0.0 1.0 0.0, limit lower=0.0 upper=1.0 effort=7.0 velocity=18.85
- added joint l_wrist_joint: type revolute, parent l_elbow_link, child l_wrist_link, origin xyz=0.0 -0.0241 -0.1822 rpy=0.0 0.0 0.0, axis 0.0 0.0 1.0, limit lower=-1.57 upper=1.57 effort=7.0 velocity=18.85
- added joint neck_joint: type revolute, parent torso, child head_link, origin xyz=0.0 0.0 0.33 rpy=0.0 0.0 0.0, axis 0.0 0.0 1.0, limit lower=-1.57 upper=1.57 effort=24.0 velocity=5.445
- added joint r_gripper_joint: type revolute, parent r_wrist_link, child r_gripper_link, origin xyz=0.0 0.0 -0.05 rpy=0.0 0.0 0.0, axis 0.0 1.0 0.0, limit lower=0.0 upper=1.0 effort=7.0 velocity=18.85
- added joint r_wrist_joint: type revolute, parent r_elbow_link, child r_wrist_link, origin xyz=0.0 0.0241 -0.1822 rpy=0.0 0.0 0.0, axis 0.0 0.0 1.0, limit lower=-1.57 upper=1.57 effort=7.0 velocity=18.85
- joint l_elbow_joint: limit lower=-2.5 upper=0.2 effort=30 velocity=10 -> lower=-2.5 upper=0.2 effort=43.0 velocity=33.51
- joint l_hip_pitch_joint: limit lower=-1.8 upper=1.2 effort=60 velocity=12 -> lower=-1.8 upper=1.2 effort=121.0 velocity=21.991
- joint l_hip_roll_joint: limit lower=-0.35 upper=0.8 effort=60 velocity=12 -> lower=-0.35 upper=0.8 effort=121.0 velocity=21.991
- joint l_knee_joint: limit lower=-0.2 upper=2.6 effort=60 velocity=12 -> lower=-0.2 upper=2.6 effort=121.0 velocity=21.991
- joint l_shoulder_pitch_joint: limit lower=-3.14 upper=3.14 effort=30 velocity=10 -> lower=-3.14 upper=3.14 effort=43.0 velocity=33.51
- joint l_shoulder_roll_joint: limit lower=-0.2 upper=2.6 effort=30 velocity=10 -> lower=-0.2 upper=2.6 effort=43.0 velocity=33.51
- joint l_shoulder_yaw_joint: limit lower=-1.57 upper=1.57 effort=30 velocity=10 -> lower=-1.57 upper=1.57 effort=43.0 velocity=33.51
- joint l_wheel_joint: limit effort=20 velocity=30 -> effort=43.0 velocity=33.51
- joint r_elbow_joint: limit lower=-2.5 upper=0.2 effort=30 velocity=10 -> lower=-2.5 upper=0.2 effort=43.0 velocity=33.51
- joint r_hip_pitch_joint: limit lower=-1.8 upper=1.2 effort=60 velocity=12 -> lower=-1.8 upper=1.2 effort=121.0 velocity=21.991
- joint r_hip_roll_joint: limit lower=-0.8 upper=0.35 effort=60 velocity=12 -> lower=-0.8 upper=0.35 effort=121.0 velocity=21.991
- joint r_knee_joint: limit lower=-0.2 upper=2.6 effort=60 velocity=12 -> lower=-0.2 upper=2.6 effort=121.0 velocity=21.991
- joint r_shoulder_pitch_joint: limit lower=-3.14 upper=3.14 effort=30 velocity=10 -> lower=-3.14 upper=3.14 effort=43.0 velocity=33.51
- joint r_shoulder_roll_joint: limit lower=-2.6 upper=0.2 effort=30 velocity=10 -> lower=-2.6 upper=0.2 effort=43.0 velocity=33.51
- joint r_shoulder_yaw_joint: limit lower=-1.57 upper=1.57 effort=30 velocity=10 -> lower=-1.57 upper=1.57 effort=43.0 velocity=33.51
- joint r_wheel_joint: limit effort=20 velocity=30 -> effort=43.0 velocity=33.51
- joint waist_pitch_joint: limit lower=-0.52 upper=0.52 effort=40 velocity=6 -> lower=-0.52 upper=0.52 effort=43.0 velocity=33.51
- joint waist_roll_joint: limit lower=-0.35 upper=0.35 effort=40 velocity=6 -> lower=-0.35 upper=0.35 effort=43.0 velocity=33.51
- joint waist_yaw_joint: limit lower=-1.57 upper=1.57 effort=30 velocity=10 -> lower=-1.57 upper=1.57 effort=43.0 velocity=33.51
